File: splitly.kicad_pcb (KiCad board)
At the start: 2 copper layers, 122 parts, among them SW1 SW_Push_45deg, SW10 SW_Push_45deg, SW11 SW_Push_45deg, SW12 SW_Push_45deg, SW13 SW_Push_45deg, SW14 SW_Push_45deg, SW15 SW_Push_45deg, SW16 SW_Push_45deg, SW17 SW_Push_45deg, SW18 SW_Push_45deg, SW19 SW_Push_45deg, SW2 SW_Push_45deg, SW20 SW_Push_45deg, SW21 SW_Push_45deg, SW22 SW_Push_45deg, SW23 SW_Push_45deg, SW24 SW_Push_45deg, SW25 SW_Push_45deg, SW26 SW_Push_45deg, SW27 SW_Push_45deg, SW28 SW_Push_45deg, SW29 SW_Push_45deg, SW3 SW_Push_45deg, SW30 SW_Push_45deg, SW31 SW_Push_45deg, SW32 SW_Push_45deg, SW33 SW_Push_45deg, SW34 SW_Push_45deg, SW35 SW_Push_45deg, SW36 SW_Push_45deg, SW37 SW_Push_45deg, SW38 SW_Push_45deg, SW39 SW_Push_45deg, SW4 SW_Push_45deg, SW40 SW_Push_45deg, SW41 SW_Push_45deg, SW42 SW_Push_45deg, SW43 SW_Push_45deg, SW44 SW_Push_45deg, SW45 SW_Push_45deg, SW46 SW_Push_45deg, SW47 SW_Push_45deg, SW48 SW_Push_45deg, SW49 SW_Push_45deg, SW5 SW_Push_45deg, SW50 SW_Push_45deg, SW51 SW_Push_45deg, SW52 SW_Push_45deg, SW53 SW_Push_45deg, SW54 SW_Push_45deg, SW55 SW_Push_45deg, SW56 SW_Push_45deg, SW57 SW_Push_45deg, SW58 SW_Push_45deg, SW59 SW_Push_45deg, SW6 SW_Push_45deg, SW60 SW_Push_45deg, SW7 SW_Push_45deg, SW8 SW_Push_45deg, SW9 SW_Push_45deg, U1 Nice_Nano_V2, U2 Nice_Nano_V2

Commit message: Made pcb + journal update :3
Parts:
- D1, D10, D11, D12, D13, D14, D15, D16, D17, D18, D19, D2, D20, D21, D22, D23, D24, D25, D26, D27, D28, D29, D3, D30, D31, D32, D33, D34, D35, D36, D37, D38, D39, D4, D40, D41, D42, D43, D44, D45, D46, D47, D48, D49, D5, D50, D51, D52, D53, D54, D55, D56, D57, D58, D59, D6, D60, D7, D8, D9: moved to B.Cu
- moved D25 280.5 mm to (32.3, 123.6), turned to 90 degrees
- moved D19 275.4 mm to (32.2, 104.7), turned to 90 degrees
- moved D13 274.9 mm to (32.6, 85.5), turned to 90 degrees
- moved D7 273.9 mm to (32.1, 66.5), turned to 90 degrees
- moved D1 273.0 mm to (32.8, 47.3), turned to 90 degrees
- moved D26 261.3 mm to (51.5, 123.7), turned to 90 degrees
- moved D20 256.6 mm to (51.4, 104.7), turned to 90 degrees
- moved D14 256.3 mm to (51.6, 85.6), turned to 90 degrees
- moved D8 255.7 mm to (51.5, 66.4), turned to 90 degrees
- moved D2 255.1 mm to (51.8, 47.3), turned to 90 degrees
- moved D27 242.0 mm to (70.7, 123.7), turned to 90 degrees
- moved D21 242.0 mm to (70.7, 104.7), turned to 90 degrees
- moved D9 237.9 mm to (70.5, 66.4), turned to 90 degrees
- moved D15 237.7 mm to (70.5, 85.6), turned to 90 degrees
- moved D3 237.4 mm to (70.8, 47.3), turned to 90 degrees
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Connections:
- D32 pad 1: /row 1 2 -> /row 0 2
- D33 pad 1: /row 2 2 -> /row 0 2
- D34 pad 1: /row 3 2 -> /row 0 2
- D35 pad 1: /row 4 2 -> /row 0 2
- D38 pad 1: /row 2 2 -> /row 1 2
- D39 pad 1: /row 3 2 -> /row 1 2
- D40 pad 1: /row 4 2 -> /row 1 2
- D41 pad 1: /row 0 2 -> /row 1 2
- D44 pad 1: /row 3 2 -> /row 2 2
- D45 pad 1: /row 4 2 -> /row 2 2
- D46 pad 1: /row 0 2 -> /row 2 2
- D47 pad 1: /row 1 2 -> /row 2 2
- D50 pad 1: /row 4 2 -> /row 3 2
- D51 pad 1: /row 0 2 -> /row 3 2
- D52 pad 1: /row 1 2 -> /row 3 2
- D53 pad 1: /row 2 2 -> /row 3 2
- D56 pad 1: /row 0 2 -> /row 4 2
- D57 pad 1: /row 1 2 -> /row 4 2
- D58 pad 1: /row 2 2 -> /row 4 2
- D59 pad 1: /row 3 2 -> /row 4 2
- SW1 pad 1: /collumn 1 -> /collumn 0
- SW2 pad 1: /collumn 2 -> /collumn 1
- SW3 pad 1: /collumn 3 -> /collumn 2
- SW32 pad 1: /collumn 0 2 -> /collumn 1 2
- SW33 pad 1: /collumn 0 2 -> /collumn 2 2
- SW34 pad 1: /collumn 0 2 -> /collumn 3 2
- SW35 pad 1: /collumn 0 2 -> /collumn 4 2
- SW36 pad 1: /collumn 1 2 -> /collumn 5 2
- SW37 pad 1: /collumn 1 2 -> /collumn 0 2
- SW39 pad 1: /collumn 1 2 -> /collumn 2 2
- SW4 pad 1: /collumn 4 -> /collumn 3
- SW40 pad 1: /collumn 1 2 -> /collumn 3 2
- SW41 pad 1: /collumn 2 2 -> /collumn 4 2
- SW42 pad 1: /collumn 2 2 -> /collumn 5 2
- SW43 pad 1: /collumn 2 2 -> /collumn 0 2
- SW44 pad 1: /collumn 2 2 -> /collumn 1 2
- SW47 pad 1: /collumn 3 2 -> /collumn 4 2
- SW48 pad 1: /collumn 3 2 -> /collumn 5 2
- SW49 pad 1: /collumn 3 2 -> /collumn 0 2
- SW5 pad 1: /collumn 5 -> /collumn 4
- SW50 pad 1: /collumn 3 2 -> /collumn 1 2
- SW51 pad 1: /collumn 4 2 -> /collumn 2 2
- SW52 pad 1: /collumn 4 2 -> /collumn 3 2
- SW54 pad 1: /collumn 4 2 -> /collumn 5 2
- SW55 pad 1: /collumn 4 2 -> /collumn 0 2
- SW56 pad 1: /collumn 5 2 -> /collumn 1 2
- SW57 pad 1: /collumn 5 2 -> /collumn 2 2
- SW58 pad 1: /collumn 5 2 -> /collumn 3 2
- SW59 pad 1: /collumn 5 2 -> /collumn 4 2
- SW6 pad 1: /collumn 0 -> /collumn 5
Routing:
- net /collumn 0: track 0.00 -> 214.2 mm
- net /collumn 1: track 0.00 -> 210.1 mm, vias 0 -> 8
- net /row 4 2: track 0.00 -> 207.0 mm
- net /row 2 2: track 0.00 -> 206.3 mm
- net /collumn 2: track 0.00 -> 190.7 mm, vias 0 -> 8
- net /row 3 2: track 0.00 -> 190.3 mm
- net /row 1 2: track 0.00 -> 187.3 mm
- net /collumn 5 2: track 0.00 -> 187.1 mm, vias 0 -> 9
- net /collumn 3: track 0.00 -> 173.8 mm, vias 0 -> 8
- net /row 4: track 0.00 -> 171.5 mm
- net /collumn 4 2: track 0.00 -> 161.9 mm, vias 0 -> 11
- net /row 3: track 0.00 -> 155.1 mm
- net /row 0 2: track 0.00 -> 152.7 mm
- net /collumn 4: track 0.00 -> 149.2 mm, vias 0 -> 8
- net /collumn 3 2: track 0.00 -> 139.5 mm, vias 0 -> 11
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Other:
- board outline added: 307.6 x 96.2 mm

Commit message: OOOOoooOOO Update
Parts:
- removed U1: Nice_Nano_V2, ScottoKeebs_MCU:Nice_Nano_V2
- added J2: Conn_02x01, Connector_JST:JST_PH_S2B-PH-K_1x02_P2.00mm_Horizontal, B.Cu at (194.3, 53.8)
- added J3: Conn_02x01, Connector_JST:JST_PH_S2B-PH-K_1x02_P2.00mm_Horizontal, B.Cu at (165.4, 53.8)
- added SW61: SW_SPDT, Button_Switch_SMD:SW_SPDT_CK_JS102011SAQN, F.Cu at (184.6, 73.9)
- added SW62: SW_SPDT, Button_Switch_SMD:SW_SPDT_CK_JS102011SAQN, F.Cu at (173.0, 74.0)
- added U3: XIAO-nRF52840-SMD, XIAO-:XIAO-nRF52840-SMD, F.Cu at (193.6, 30.5)
- SW1, SW10, SW11, SW12, SW13, SW14, SW15, SW16, SW17, SW18, SW19, SW2, SW20, SW21, SW22, SW23, SW24, SW25, SW26, SW27, SW28, SW29, SW3, SW30, SW31, SW32, SW33, SW34, SW35, SW36, SW37, SW38, SW39, SW4, SW40, SW41, SW42, SW43, SW44, SW45, SW46, SW47, SW48, SW49, SW5, SW50, SW51, SW52, SW53, SW54, SW55, SW56, SW57, SW58, SW59, SW6, SW60, SW7, SW8, SW9: footprint Kailh_PG1353_Hotswap:Kailh-PG1353-Hotswap-1U -> ScottoKeebs_Hotswap:Hotswap_Choc_V1_1.00u; moved to F.Cu
- U2: value Nice_Nano_V2 -> XIAO-nRF52840-SMD; footprint ScottoKeebs_MCU:Nice_Nano_V2 -> XIAO-:XIAO-nRF52840-SMD
- moved D25 40.0 mm to (63.1, 98.0)
- moved D26 39.5 mm to (81.4, 97.9)
- moved D19 39.1 mm to (62.9, 80.5)
- moved D20 38.4 mm to (81.1, 80.5)
- moved D27 38.3 mm to (99.2, 98.1)
- moved D13 37.8 mm to (63.0, 63.1)
- moved U2 37.7 mm to (164.2, 30.5)
- moved D21 37.3 mm to (99.2, 80.6)
- moved D28 37.3 mm to (117.2, 98.1)
- moved D29 37.0 mm to (135.4, 98.0)
- moved D7 37.0 mm to (63.0, 46.2)
- moved D22 36.9 mm to (117.5, 80.4)
- moved D14 36.7 mm to (81.0, 63.7)
- moved D15 36.3 mm to (99.1, 63.3)
- moved D30 36.1 mm to (153.4, 98.0)
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Connections:
- U2 pad 1: unconnected-(U2-Pad1) -> /row 0
- U2 pad 10: unconnected-(U2-7-Pad10) -> /collumn 3
- U2 pad 11: unconnected-(U2-8-Pad11) -> /collumn 2
- U2 pad 13: unconnected-(U2-10-Pad13) -> GND
- U2 pad 15: /collumn 5 2 -> Net-(SW62-B)
- U2 pad 16: /collumn 4 2 -> GND
- U2 pad 17: /collumn 3 2 -> unconnected-(U2-NFC1-Pad17)
- U2 pad 18: /collumn 2 2 -> unconnected-(U2-NFC2-Pad18)
- U2 pad 19: /collumn 1 2 -> unconnected-(U2-PA31_SWDIO-Pad19)
- U2 pad 2: /row 0 2 -> /row 1
- U2 pad 20: /collumn 0 2 -> unconnected-(U2-PA30_SWCLK-Pad20)
- U2 pad 22: unconnected-(U2-RST-Pad22) -> GND
- U2 pad 3: unconnected-(U2-GND-Pad3) -> /row 2
- U2 pad 4: unconnected-(U2-GND-Pad4) -> /row 3
- U2 pad 5: /row 1 2 -> /row 4
- U2 pad 6: /row 2 2 -> /collumn 0
- U2 pad 7: /row 3 2 -> /collumn 1
- U2 pad 8: /row 4 2 -> /collumn 5
- U2 pad 9: unconnected-(U2-6-Pad9) -> /collumn 4
Routing:
- net Net-(SW62-B): track 0.00 -> 52.5 mm
- net Net-(SW61-B): track 0.00 -> 44.6 mm
- net GND1: track 0.00 -> 42.3 mm
- net GND: track 0.00 -> 42.3 mm
- net /row 2 2: track 206.3 -> 165.3 mm, vias 0 -> 12
- net /row 1 2: track 187.3 -> 147.4 mm, vias 0 -> 13
- net /collumn 3: track 173.8 -> 136.1 mm, vias 8 -> 3
- net /collumn 2: track 190.7 -> 154.9 mm, vias 8 -> 3
- net /collumn 4: track 149.2 -> 118.7 mm, vias 8 -> 3
- net Net-(J3-Pin_1): track 0.00 -> 29.7 mm
- net /collumn 1: track 210.1 -> 180.6 mm, vias 8 -> 3
- net /collumn 5: track 130.4 -> 101.5 mm, vias 8 -> 1
- net Net-(J2-Pin_1): track 0.00 -> 27.3 mm
- net /collumn 0: track 214.2 -> 195.2 mm, vias 0 -> 1
- net /collumn 5 2: track 187.1 -> 169.1 mm, vias 9 -> 1
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- added copper zone on B.Cu, net (none)
- added copper zone on F.Cu, net (none)
Other:
- board size 307.6 x 96.2 mm -> 271.5 x 85.6 mm

Commit message: :yay:
Parts:
- removed J2, J3: Conn_02x01, Connector_JST:JST_PH_S2B-PH-K_1x02_P2.00mm_Horizontal
- removed SW61, SW62: SW_SPDT, Button_Switch_SMD:SW_SPDT_CK_JS102011SAQN
- removed U3: XIAO-nRF52840-SMD, XIAO-:XIAO-nRF52840-SMD
- added U1: XIAO-nRF52840-DIP, XIAO-:XIAO-nRF52840-DIP, F.Cu at (193.4, 30.6)
- U2: value XIAO-nRF52840-SMD -> XIAO-nRF52840-DIP; footprint XIAO-:XIAO-nRF52840-SMD -> XIAO-:XIAO-nRF52840-DIP
- moved U2 0.37 mm to (164.5, 30.5)
Routing:
- net Net-(SW62-B): track 52.5 -> 0.00 mm
- net Net-(SW61-B): track 44.6 -> 0.00 mm
- net GND1: track 42.3 -> 0.00 mm
- net GND: track 42.3 -> 0.00 mm
- net Net-(J3-Pin_1): track 29.7 -> 0.00 mm
- net Net-(J2-Pin_1): track 27.3 -> 0.00 mm
- net /row 1 2: track 147.4 -> 160.9 mm, vias 13 -> 12
- net /row 2 2: track 165.3 -> 171.3 mm, vias 12 -> 11
- net /row 2: track 133.8 -> 139.1 mm
- net /row 4 2: track 189.2 -> 194.2 mm, vias 11 -> 10
- net /row 0 2: track 142.4 -> 147.2 mm
- net /collumn 0: track 195.2 -> 197.7 mm, vias 1 -> 2
- net /collumn 0 2: track 96.6 -> 98.8 mm
- net /row 3 2: track 182.1 -> 179.9 mm, vias 11 -> 12
- net /collumn 5 2: track 169.1 -> 171.1 mm
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