File: splitly.kicad_sch (KiCad schematic)
At the start: 122 parts, among them SW1 SW_Push_45deg, SW10 SW_Push_45deg, SW11 SW_Push_45deg, SW12 SW_Push_45deg, SW13 SW_Push_45deg, SW14 SW_Push_45deg, SW15 SW_Push_45deg, SW16 SW_Push_45deg, SW17 SW_Push_45deg, SW18 SW_Push_45deg, SW19 SW_Push_45deg, SW2 SW_Push_45deg, SW20 SW_Push_45deg, SW21 SW_Push_45deg, SW22 SW_Push_45deg, SW23 SW_Push_45deg, SW24 SW_Push_45deg, SW25 SW_Push_45deg, SW26 SW_Push_45deg, SW27 SW_Push_45deg, SW28 SW_Push_45deg, SW29 SW_Push_45deg, SW3 SW_Push_45deg, SW30 SW_Push_45deg, SW31 SW_Push_45deg, SW32 SW_Push_45deg, SW33 SW_Push_45deg, SW34 SW_Push_45deg, SW35 SW_Push_45deg, SW36 SW_Push_45deg, SW37 SW_Push_45deg, SW38 SW_Push_45deg, SW39 SW_Push_45deg, SW4 SW_Push_45deg, SW40 SW_Push_45deg, SW41 SW_Push_45deg, SW42 SW_Push_45deg, SW43 SW_Push_45deg, SW44 SW_Push_45deg, SW45 SW_Push_45deg, SW46 SW_Push_45deg, SW47 SW_Push_45deg, SW48 SW_Push_45deg, SW49 SW_Push_45deg, SW5 SW_Push_45deg, SW50 SW_Push_45deg, SW51 SW_Push_45deg, SW52 SW_Push_45deg, SW53 SW_Push_45deg, SW54 SW_Push_45deg, SW55 SW_Push_45deg, SW56 SW_Push_45deg, SW57 SW_Push_45deg, SW58 SW_Push_45deg, SW59 SW_Push_45deg, SW6 SW_Push_45deg, SW60 SW_Push_45deg, SW7 SW_Push_45deg, SW8 SW_Push_45deg, SW9 SW_Push_45deg, U1 Nice_Nano_V2, U2 Nice_Nano_V2

Commit message: Made pcb + journal update :3
Parts:
- renumbered D6 to D1, D1 to D2, D2 to D3, D36 to D32, D41 to D33, D46 to D34, D51 to D35, D56 to D36, D32 to D37, D37 to D38, D42 to D39, D3 to D4, D47 to D40, D52 to D41, D57 to D42, D33 to D43, D38 to D44, D43 to D45, D48 to D46, D53 to D47, D58 to D48, D34 to D49, D4 to D5, D39 to D50, D44 to D51, D49 to D52, D54 to D53, D59 to D54, D35 to D55, D40 to D56, D45 to D57, D50 to D58, D55 to D59, D5 to D6, SW6 to SW1, SW1 to SW2, SW2 to SW3, SW36 to SW32, SW41 to SW33, SW46 to SW34, SW51 to SW35, SW56 to SW36, SW32 to SW37, SW37 to SW38, SW42 to SW39, SW3 to SW4, SW47 to SW40, SW52 to SW41, SW57 to SW42, SW33 to SW43, SW38 to SW44, SW43 to SW45, SW48 to SW46, SW53 to SW47, SW58 to SW48, SW34 to SW49, SW4 to SW5, SW39 to SW50, SW44 to SW51, SW49 to SW52, SW54 to SW53, SW59 to SW54, SW35 to SW55, SW40 to SW56, SW45 to SW57, SW50 to SW58, SW55 to SW59, SW5 to SW6

Commit message: OOOOoooOOO Update
Parts:
- removed U1, U2: Nice_Nano_V2, ScottoKeebs_MCU:Nice_Nano_V2, symbol ScottoKeebs:MCU_Nice_Nano_V2
- added J2, J3: Conn_02x01, Connector_JST:JST_PH_S2B-PH-K_1x02_P2.00mm_Horizontal, symbol Connector_Generic:Conn_02x01
- added SW61, SW62: SW_SPDT, Button_Switch_SMD:SW_SPDT_CK_JS102011SAQN, symbol Switch:SW_SPDT
- added U2, U3: XIAO-nRF52840-SMD, XIAO-:XIAO-nRF52840-SMD, symbol Seeed_Studio_XIAO_Series:XIAO-nRF52840-SMD
- SW1, SW10, SW11, SW12, SW13, SW14, SW15, SW16, SW17, SW18, SW19, SW2, SW20, SW21, SW22, SW23, SW24, SW25, SW26, SW27, SW28, SW29, SW3, SW30, SW31, SW32, SW33, SW34, SW35, SW36, SW37, SW38, SW39, SW4, SW40, SW41, SW42, SW43, SW44, SW45, SW46, SW47, SW48, SW49, SW5, SW50, SW51, SW52, SW53, SW54, SW55, SW56, SW57, SW58, SW59, SW6, SW60, SW7, SW8, SW9: footprint Kailh_PG1353_Hotswap:Kailh-PG1353-Hotswap-1U -> ScottoKeebs_Hotswap:Hotswap_Choc_V1_1.00u
Connections:
- net collumn 0: now also U2.6 (P0.05_A5_D5_SCL)
- net collumn 0 2: now also U3.6 (P0.05_A5_D5_SCL)
- net collumn 1: now also U2.7 (P1.11_D6_TX)
- net collumn 1 2: now also U3.7 (P1.11_D6_TX)
- net collumn 2: now also U2.11 (P1.15_D10_MOSI)
- net collumn 2 2: now also U3.11 (P1.15_D10_MOSI)
- net collumn 3: now also U2.10 (P1.14_D9_MISO)
- net collumn 3 2: now also U3.10 (P1.14_D9_MISO)
- net collumn 4: now also U2.9 (P1.13_D8_SCK)
- net collumn 4 2: now also U3.9 (P1.13_D8_SCK)
- net collumn 5: now also U2.8 (P1.12_D7_RX)
- net collumn 5 2: now also U3.8 (P1.12_D7_RX)
- net row 0: now also U2.1 (P0.02_A0_D0)
- net row 0 2: now also U3.1 (P0.02_A0_D0)
- net row 1: now also U2.2 (P0.03_A1_D1)
- net row 1 2: now also U3.2 (P0.03_A1_D1)
- net row 2: now also U2.3 (P0.28_A2_D2)
- net row 2 2: now also U3.3 (P0.28_A2_D2)
- net row 3: now also U2.4 (P0.29_A3_D3)
- net row 3 2: now also U3.4 (P0.29_A3_D3)
- net row 4: now also U2.5 (P0.04_A4_D4_SDA)
- net row 4 2: now also U3.5 (P0.04_A4_D4_SDA)
- new net: SW61.2 (B), U3.15 (BAT)
- new net: J2.1 (Pin_1), SW61.3 (C)
- new net: J3.1 (Pin_1), SW62.3 (C)
- new net: SW62.2 (B), U2.15 (BAT)
- new net GND: J3.2 (Pin_2), U2.13 (GND), U2.16 (GND), U2.22 (GND)
- new net GND1: J2.2 (Pin_2), U3.13 (GND), U3.16 (GND), U3.22 (GND)

Commit message: :yay:
Parts:
- removed J2, J3: Conn_02x01, Connector_JST:JST_PH_S2B-PH-K_1x02_P2.00mm_Horizontal, symbol Connector_Generic:Conn_02x01
- removed SW61, SW62: SW_SPDT, Button_Switch_SMD:SW_SPDT_CK_JS102011SAQN, symbol Switch:SW_SPDT
- removed U2, U3: XIAO-nRF52840-SMD, XIAO-:XIAO-nRF52840-SMD, symbol Seeed_Studio_XIAO_Series:XIAO-nRF52840-SMD
- added U1, U2: XIAO-nRF52840-DIP, XIAO-:XIAO-nRF52840-DIP, symbol Seeed_Studio_XIAO_Series:XIAO-nRF52840-DIP
Connections:
- net GND: now also U2.13 (GND)
- net GND1: now also U1.13 (GND)
- net collumn 0: now also U2.6 (P0.05_AIN3_A5_D5)
- net collumn 0 2: now also U1.6 (P0.05_AIN3_A5_D5)
- net collumn 1: now also U2.7 (P1.11_TX_D6)
- net collumn 1 2: now also U1.7 (P1.11_TX_D6)
- net collumn 2: now also U2.11 (P1.15_MOSI_D10)
- net collumn 2 2: now also U1.11 (P1.15_MOSI_D10)
- net collumn 3: now also U2.10 (P1.14_MISO_D9)
- net collumn 3 2: now also U1.10 (P1.14_MISO_D9)
- net collumn 4: now also U2.9 (P1.13_SCK_D8)
- net collumn 4 2: now also U1.9 (P1.13_SCK_D8)
- net collumn 5: now also U2.8 (P1.12_RX_D7)
- net collumn 5 2: now also U1.8 (P1.12_RX_D7)
- net row 0: now also U2.1 (P0.02_AIN0_LOW_A0_D0)
- net row 0 2: now also U1.1 (P0.02_AIN0_LOW_A0_D0)
- net row 1: now also U2.2 (P0.03_AIN1_LOW_A1_D1)
- net row 1 2: now also U1.2 (P0.03_AIN1_LOW_A1_D1)
- net row 2: now also U2.3 (P0.28_AIN4_LOW_A2_D2)
- net row 2 2: now also U1.3 (P0.28_AIN4_LOW_A2_D2)
- net row 3: now also U2.4 (P0.29_AIN5_LOW_A3_D3)
- net row 3 2: now also U1.4 (P0.29_AIN5_LOW_A3_D3)
- net row 4: now also U2.5 (P0.04_AIN2_A4_D4)
- net row 4 2: now also U1.5 (P0.04_AIN2_A4_D4)
